File: blinkencontrol/blinkencontrol.sch (EAGLE design)
At the start: 21 parts, among them IC1 AT90S2313P, IC2 7805TV, Q1 20MHz, T1 BC337, T2 BC337, T3 BC337

Commit message: blinkencontrol: Fix C1/C2 value
Parts:
- C1, C2: value 22nF -> 22pF
Changed lines of the file:
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@@
 <part name="R4" library="resistor" deviceset="R-EU_" device="0207/10" value="1k"/>
 <part name="R5" library="resistor" deviceset="R-EU_" device="0207/10" value="1k"/>
-<part name="C1" library="capacitor-wima" deviceset="C" device="2.5/2" value="22nF"/>
-<part name="C2" library="capacitor-wima" deviceset="C" device="2.5/2" value="22nF"/>
+<part name="C1" library="capacitor-wima" deviceset="C" device="2.5/2" value="22pF"/>
+<part name="C2" library="capacitor-wima" deviceset="C" device="2.5/2" value="22pF"/>
 <part name="T1" library="transistor" deviceset="*-NPN-" device="TO92-CBE" technology="BC337-40" value="BC337"/>
 <part name="T2" library="transistor" deviceset="*-NPN-" device="TO92-CBE" technology="BC337-40" value="BC337"/>
