File: avrshift/avrshift.brd (EAGLE design)
At the start: 60.6 x 69.8 mm, 56 parts, among them IC1 AT90S2313P, IC2 7805TV, Q1 BC337-40, Q10 BC337-40, Q11 BC337-40, Q12 BC337-40, Q13 BC337-40, Q2 BC337-40, Q3 BC337-40, Q4 BC337-40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

Commit message: avrshift: schematic/baord bugfixes
Parts:
- LED1: value LINK -> PWR
Changed lines of the file:
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@@
 <element name="R15" library="resistor" package="0207/10" value="470" x="15.24" y="41.91"/>
 <element name="R18" library="resistor" package="0207/10" value="470" x="15.24" y="46.99"/>
-<element name="LED1" library="led" package="LED3MM" value="LINK" x="6.35" y="41.91" rot="R180"/>
+<element name="LED1" library="led" package="LED3MM" value="PWR" x="6.35" y="41.91" rot="R180"/>
 <element name="LED2" library="led" package="LED3MM" value="ACT" x="6.35" y="46.99" rot="R180"/>
 <element name="JP1" library="pinhead" package="1X02" value="" x="10.16" y="64.77" rot="R180"/>
