File: avrshift/avrshift-uln2803.brd (EAGLE design)
At the start: 49.2 x 49.5 mm, 32 parts, among them IC1 AT90S2313P, IC2 7805TV

Commit message: some more minor adjustments (especially labels)
Parts:
- IC3, IC4: value (none) -> ULN2803A

Commit message: wat
Parts:
- moved JP2 21.6 mm to (45.7, 45.7), turned to 270 degrees
- moved SJ2 8.89 mm to (5.08, 14.0)
- moved R1 6.48 mm to (16.5, 12.7), turned to 180 degrees
- moved R2 6.35 mm to (12.7, 14.0)
- moved R3 4.58 mm to (17.8, 44.5)
- moved C2 4.02 mm to (22.9, 44.5), turned to 270 degrees
- moved JP3 2.54 mm to (41.9, 44.5)
- moved R18 1.80 mm to (12.7, 35.6)
- moved R15 1.27 mm to (12.7, 31.8)
Routing:
- net BUSGND: track 41.5 -> 25.0 mm
- net VCC: track 91.3 -> 98.0 mm
- net N$4: track 4.34 -> 10.7 mm
- net SCL: track 5.61 -> 11.7 mm
- net N$2: track 13.2 -> 7.62 mm
- net N$1: track 4.34 -> 8.67 mm
- net 5V: track 16.6 -> 20.9 mm
- net N$5: track 5.08 -> 2.54 mm
- net SDA: track 9.72 -> 11.7 mm
- net N$8: track 2.54 -> 4.34 mm
- net N$21: track 7.93 -> 6.13 mm
- net N$33: track 6.13 -> 4.86 mm
- net N$3: track 2.54 -> 3.81 mm
- net N$10: track 2.54 -> 3.81 mm
