File: avrshift/avrshift-uln2803.brd (EAGLE design)
At the start: 49.2 x 49.5 mm, 32 parts, among them IC1 AT90S2313P, IC2 7805TV, IC3 ULN2803A, IC4 ULN2803A

Commit message: 😺
Parts:
- C2: device capacitor-wima:C2.5-3 -> rcl:C050-024X044
- turned C2 to 180 degrees
Routing:
- net 5V: track 20.9 -> 21.7 mm
- net AVRO02: track 18.4 -> 17.7 mm
Other:
- board text added: "avrshift"
- board text added: "dorfmap"
- board text added: "rev 2"

Commit message: avrshift-uln2803: start work on rev 2.1
Parts:
- added SV2: (no value), pinhead:2X03
- moved LED2 31.2 mm to (25.4, 12.1), turned to 0 degrees
- moved LED1 30.7 mm to (25.4, 7.62), turned to 0 degrees
- moved R18 24.1 mm to (20.3, 12.7)
- moved R15 19.2 mm to (15.2, 12.7)
- moved R2 7.73 mm to (5.08, 12.7), turned to 0 degrees
- moved SJ1 6.98 mm to (2.54, 21.0)
- moved SJ2 6.98 mm to (5.08, 21.0)
- moved R1 6.35 mm to (10.2, 12.7), turned to 0 degrees
- moved OK1 2.62 mm to (13.3, 20.3)
- moved OK2 2.62 mm to (6.99, 20.3)
- moved C2 0.64 mm to (23.5, 44.5)
- moved IC1 0.64 mm to (22.2, 27.9)
- moved R3 0.64 mm to (17.1, 44.5), turned to 180 degrees
Connections:
- removed net N$3: IC1.1, R3.2
- new net RST: IC1.1, R3.1, SV2.5
- net 5V: now also R3.2, SV2.2; no longer R3.1
- net AVRO11: now also SV2.4
- net AVRO12: now also SV2.1
- net AVRO13: now also SV2.3
- net GND: now also SV2.6
- net N$10: now also R15.2; no longer R15.1
- net N$21: now also R18.1; no longer R18.2
- net N$33: now also R15.1; no longer R15.2
- net N$8: now also R18.2; no longer R18.1
Routing:
- net AVRO12: track 7.18 -> 30.8 mm
- net AVRO11: track 7.18 -> 29.0 mm, vias 0 -> 1
- net N$33: track 4.86 -> 24.9 mm, vias 0 -> 1
- net AVRO13: track 7.93 -> 27.3 mm
- net RST: track 0.00 -> 19.0 mm
- net N$21: track 6.13 -> 21.3 mm
- net BUSGND: track 25.0 -> 37.7 mm
- net 5V: track 21.7 -> 33.9 mm
- net BUSVCC: track 7.17 -> 15.0 mm
- net VCC: track 98.0 -> 91.0 mm
- net SCL: track 11.7 -> 5.08 mm
- net N$10: track 3.81 -> 10.5 mm
- net N$4: track 10.7 -> 4.07 mm
- net N$1: track 8.67 -> 4.07 mm
- net N$3: track 3.81 -> 0.00 mm
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Other:
- board text added: "1"
- board text added: "ISP"
- board text added: "SI2C"
- board text added: "derf"
- board text added: "rev 2.1"
- board text removed: "rev 2"
