File: client/hub/hub.sch (EAGLE design)
At the start: 12 parts

Commit message: hub: bigger solder pads for the damn connectors
Parts:
- SV1, SV2, SV3, SV4: device con-harting-ml:ML10 -> con-harting-ml-derf:ML10
Changed lines of the file:
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@@
 </classes>
 <parts>
-<part name="SV1" library="con-harting-ml" deviceset="ML10" device="" value="SI2C"/>
+<part name="SV1" library="con-harting-ml-derf" deviceset="ML10" device="" value="SI2C"/>
 <part name="JP1" library="pinhead" deviceset="PINHD-1X2" device="" value="PWR"/>
-<part name="SV2" library="con-harting-ml" deviceset="ML10" device="" value="SI2C"/>
-<part name="SV3" library="con-harting-ml" deviceset="ML10" device="" value="SI2C"/>
-<part name="SV4" library="con-harting-ml" deviceset="ML10" device="" value="SI2C"/>
+<part name="SV2" library="con-harting-ml-derf" deviceset="ML10" device="" value="SI2C"/>
+<part name="SV3" library="con-harting-ml-derf" deviceset="ML10" device="" value="SI2C"/>
+<part name="SV4" library="con-harting-ml-derf" deviceset="ML10" device="" value="SI2C"/>
 <part name="JP2" library="pinhead" deviceset="PINHD-1X2" device="" value="DATA"/>
 <part name="H1" library="holes" deviceset="MOUNT-HOLE" device="3.2" value="MOUNT-HOLE3.2"/>
